Commit message: collision tracking trials
did major changes, collision tracking still not implemented

File: Gazebo/urdf/quadrotor_base.urdf.xacro (robot description, xacro)
@@ -22,4 +22,17 @@
         </geometry>
       </collision>
+<!--
+      <gazebo reference="base_link">
+        <sensor type="contact" name="base_link_contact_sensor">
+          <contact>
+            <collision>base_link_collision</collision>
+          </contact>
+          <plugin name="gazebo_ros_bumper_controller" filename="libgazebo_ros_bumper.so">
+            <frameName>base_link</frameName>
+            <bumperTopicName>collision</bumperTopicName>
+            <updateRate>100.0</updateRate>
+          </plugin>
+        </sensor>
+      </gazebo> -->
     </link>
   </xacro:macro>

File: Gazebo/urdf/sensors/quadrotor_sensors.urdf.xacro (robot description, xacro)
@@ -57,4 +57,18 @@
         <frameName>map</frameName>
       </plugin>
+      <!-- <plugin name="quadrotor_contact_sensor" filename="libgazebo_ros_bumper.so">
+        <alwaysOn>true</alwaysOn>
+        <updateRate>100.0</updateRate>
+        <bodyName>base_link</bodyName>
+        <topicName>/${robot_name}/bumperTopic</topicName>
+        <bumperTopic>/${robot_name}/collision</bumperTopic>
+        <collisionTopic>/${robot_name}/collision</collisionTopic>
+      </plugin> -->
+      <plugin name="gazebo_ros_bumper_controller" filename="libgazebo_ros_bumper.so">
+        <alwaysOn>true</alwaysOn>
+        <updateRate>100.0</updateRate>
+        <frameName>base_link</frameName>
+        <bumperTopicName>/${robot_name}/collision</bumperTopicName>
+      </plugin>
     </gazebo>
   </xacro:macro>
